File: arm_20to10.kicad_pcb (KiCad board)
At the start: 2 copper layers, 16.9 x 29.7 mm, 10 parts, among them J1 SFH11-PBPC-D10-RA-BK, J2 20021111-00010T4LF, SW1 SSSS810701, U1 MIC5504-3.3YM5 TR

Commit message: Updated Kicad project files for v2.2 build of board. Add my custom library as a submodule. Probably messed up some git commands
Parts:
- added J3: CONN_02X05, Pin_Headers:Pin_Header_Straight_2x05, F.Cu at (140.3, 95.2)
- added J4: CONN_02X05, kicadlib:ARM_10_PIN_SMT, F.Cu at (150.6, 103.6)
- added J5: CONN_02X05, Pin_Headers:Pin_Header_Straight_2x05, F.Cu at (134.6, 118.7)
- added J6: CONN_02X03, Pin_Headers:Pin_Header_Straight_2x03, F.Cu at (151.6, 117.5)
- J2: value 20021111-00010T4LF -> CONN_02X10; footprint kicadlib:ARM_10_PIN -> kicadlib:ARM_20_PIN_SMT
- SW1: value SSSS810701 -> SS-12D07-VG; footprint kicadlib:SWITCH_SLIDE_SSSS810701 -> kicadlib:SS-12D07-VG-kes
- moved C2 105.0 mm to (125.1, 115.6)
- moved U1 103.4 mm to (125.1, 118.1)
- moved J2 103.1 mm to (132.7, 98.6), turned to 270 degrees
- moved D2 102.5 mm to (125.1, 95.2), turned to 0 degrees
- moved C1 101.7 mm to (123.2, 119.4), turned to 270 degrees
- moved J1 101.4 mm to (120.7, 95.2)
- moved D1 99.9 mm to (125.1, 113.7), turned to 0 degrees
- moved R2 99.9 mm to (127.0, 95.2), turned to 90 degrees
- moved R1 99.4 mm to (128.3, 112.4), turned to 90 degrees
- moved SW1 86.1 mm to (150.5, 91.4)
Connections:
- C2 pad 1: Net-(C2-Pad1) -> /LDO_OUT
- C2 pad 2: Net-(C2-Pad2) -> GND
- D1 pad 1: /5V -> Net-(D1-Pad1)
- D1 pad 2: Net-(D1-Pad2) -> /5V
- D2 pad 1: /VCC -> Net-(D2-Pad1)
- D2 pad 2: Net-(D2-Pad2) -> /VCC
- J2 pad 7: /RTCK -> Net-(J2-Pad7)
- R1 pad 2: Net-(D1-Pad2) -> Net-(D1-Pad1)
- R2 pad 2: Net-(D2-Pad2) -> Net-(D2-Pad1)
- SW1 pad 2: Net-(SW1-Pad2) -> /LDO_OUT
- U1 pad 5: Net-(SW1-Pad2) -> /LDO_OUT
Routing:
- net /TMS/SWDIO: track 11.3 -> 95.1 mm, vias 1 -> 0
- net /TCLK/SWCLK: track 14.6 -> 82.2 mm, vias 0 -> 3
- net /LDO_OUT: track 0.00 -> 63.4 mm
- net /SWO/TDO: track 14.9 -> 73.3 mm, vias 0 -> 2
- net /NRST: track 11.3 -> 56.4 mm, vias 1 -> 2
- net GND: track 0.00 -> 30.7 mm, vias 0 -> 6
- net /VCC: track 19.8 -> 50.0 mm, vias 1 -> 14
- net Net-(SW1-Pad2): track 23.7 -> 0.00 mm
- net /RTCK: track 8.13 -> 30.9 mm, vias 0 -> 2
- net /TDI: track 23.1 -> 39.5 mm, vias 0 -> 4
- net Net-(D1-Pad1): track 0.00 -> 3.70 mm
- net /5V: track 16.7 -> 13.4 mm
- net Net-(D1-Pad2): track 2.03 -> 0.00 mm
- net Net-(D2-Pad1): track 0.00 -> 1.91 mm
- net Net-(D2-Pad2): track 1.78 -> 0.00 mm
- added copper zone on F.Cu, net /VCC
- removed copper zone on F.Cu, net GND
Other:
- board size 16.9 x 29.7 mm -> 40.1 x 35.6 mm
- net class Default: clearance 0.254 -> 0.2032; trace_width 0.254 -> 0.2032; via_dia 0.889 -> 0.434; via_drill 0.635 -> 0.31
- net class Power added: clearance 0.254, trace_width 0.254, via_dia 0.889, via_drill 0.635
- rule trace_clearance: 0.254 -> 0.2032
- rule trace_min: 0.1524 -> 0.16
- rule via_min_drill: 0.33 -> 0.31
- rule via_min_size: 0.508 -> 0.31
- board text added: "1"
- board text added: "10"
- board text added: "2"
- board text added: "9"
- board text added: "APC STM32 PRG"
- board text added: "EXT PWR"
- board text added: "HOST"
- board text added: "ON"
- board text added: "Original design by Noah P."
- board text added: "TARGET"
- board text added: "github.com/kesyog/arm_20to10 v2.2"
- board text removed: "<HOST"
- board text removed: "ON|OFF"
- board text removed: "TRGT>"
- board text removed: "github.com/noahp/arm_20to10 v2.1"
