File: arm_20to10.sch (KiCad schematic (older format))
At the start: 10 parts, among them J1 SFH11-PBPC-D10-RA-BK, J2 20021111-00010T4LF, SW1 SSSS810701, U1 MIC5504-3.3YM5 TR

Commit message: Updated Kicad project files for v2.2 build of board. Add my custom library as a submodule. Probably messed up some git commands
Parts:
- removed J2: 20021111-00010T4LF, kicadlib:ARM_10_PIN, symbol ARM_10PIN
- added J2: CONN_02X10, kicadlib:ARM_20_PIN_SMT, symbol CONN_02X10
- added J3, J5: CONN_02X05, Pin_Headers:Pin_Header_Straight_2x05, symbol CONN_02X05
- added J4: CONN_02X05, kicadlib:ARM_10_PIN_SMT, symbol CONN_02X05
- added J6: MF-CON-2.54mm-2x3, Pin_Headers:Pin_Header_Straight_2x03, symbol CONN_02X03
- J1: Distrib Link (none) -> http://www.digikey.com/product-detail/en/SFH11-PBPC-D10-RA-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; Distrib PN (none) -> S9205-ND; MFG Name (none) -> Sullins; MFG PN (none) -> SFH11-PBPC-D10-RA-BK
- SW1: value SSSS810701 -> OS102011MA1QS1; footprint kicadlib:SWITCH_SLIDE_SSSS810701 -> kicadlib:SS-12D07-VG-kes; Distrib Link (none) -> http://www.digikey.com/product-detail/en/c-k-components/SS-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; Distrib PN (none) -> CKN10397-ND; MFG Name (none) -> C&K; MFG PN (none) -> SS-12D07-VG 4 NS GA PA
Connections:
- net labels added: LDO_OUT
- wire segments 52 -> 97
- no-connect marks 3 -> 14
Other:
- note added: "10-pin Cortex\nSMT connector"
- note added: "10-pin Cortex\nthrough-hole connector"
- note added: "10-pin unknown\nthrough-hole connector"
- note added: "20-pin SMT Cortex\nDebug+ETM connector"
- note added: "20-pin right angle connector\n(to debugger)"
- note added: "Amarok connector"
